Commit message: add

File: src/hector_models/hector_sensors_description/urdf/asus_camera.urdf.xacro (robot description, xacro)
@@ -13,5 +13,4 @@
       </joint>
       <link name="${name}_link">
-      <!--  commented b/c it makes quad unstable in gazebo when sending cmd_vel commands 19-01-2024
         <inertial>
           <mass value="0.200" />
@@ -19,5 +18,4 @@
           <inertia ixx="5.8083e-4" ixy="0" ixz="0" iyy="3.0833e-5" iyz="0" izz="5.9083e-4" />
         </inertial>
-        -->
         <visual>
           <origin xyz="0 0 0" rpy="0 0 0" />

File: src/hector_quadrotor/hector_quadrotor_description/urdf/quadrotor_base.urdf.xacro (robot description, xacro)
@@ -1,5 +1,5 @@
 <?xml version="1.0"?>
 <robot xmlns:xacro="http://www.ros.org/wiki/xacro">
-  <!-- <xacro:include filename="$(find hector_sensors_description)/urdf/sonar_sensor.urdf.xacro" /> -->
+  <xacro:include filename="$(find hector_sensors_description)/urdf/sonar_sensor.urdf.xacro" />
   <xacro:property name="pi" value="3.1415926535897931" />
   <!-- Main quadrotor link -->
@@ -25,7 +25,7 @@
     </link>
     <!-- Sonar height sensor -->
-    <!-- <xacro:sonar_sensor name="sonar" parent="base_link" ros_topic="sonar_height" update_rate="10" min_range="0.03" max_range="3.0" field_of_view="${40*pi/180}" ray_count="3">
+    <xacro:sonar_sensor name="sonar" parent="base_link" ros_topic="sonar_height" update_rate="10" min_range="0.03" max_range="3.0" field_of_view="${40*pi/180}" ray_count="3">
       <origin xyz="-0.16 0.0 -0.012" rpy="0 ${90*pi/180} 0"/>
-    </xacro:sonar_sensor> -->
+    </xacro:sonar_sensor>
   </xacro:macro>
 </robot>

File: src/hector_quadrotor/hector_quadrotor_description/urdf/quadrotor_with_asus.urdf.xacro (robot description, xacro)
@@ -9,5 +9,5 @@
     <xacro:include filename="$(find hector_sensors_description)/urdf/asus_camera.urdf.xacro" />
     <xacro:asus_camera name="camera" parent="base_link">
-      <origin xyz="0.1 0.0 -0.03" rpy="0 ${M_PI/9} 0"/>  <!-- PI/9  -->
+      <origin xyz="0.1 0.0 -0.03" rpy="0 ${M_PI/9} 0"/>
     </xacro:asus_camera>
 </robot>

File: src/hector_quadrotor/hector_quadrotor_description/urdf/quadrotor_with_asus_with_hokuyo_utm30lx.urdf.xacro (robot description, xacro)
@@ -14,5 +14,5 @@
     <xacro:include filename="$(find hector_sensors_description)/urdf/asus_camera.urdf.xacro" />
     <xacro:asus_camera name="camera" parent="base_link">
-      <origin xyz="0.1 0.0 -0.03" rpy="0 ${M_PI/2} 0"/>  <!-- PI/9 -->
+      <origin xyz="0.1 0.0 -0.03" rpy="0 ${M_PI/9} 0"/> <!-- changed from {M_PI/2} -->
     </xacro:asus_camera>
 </robot>

File: src/hector_quadrotor/hector_quadrotor_gazebo/urdf/quadrotor_sensors.gazebo.xacro (robot description, xacro)
@@ -16,5 +16,4 @@
             <rateGaussianNoise>0.05 0.05 0.015</rateGaussianNoise>
           </plugin>
-          <!--   now requied for now
           <plugin name="quadrotor_baro_sim" filename="libhector_gazebo_ros_baro.so">
             <updateRate>10.0</updateRate>
@@ -56,5 +55,4 @@
             <frameName>$(arg world_frame)</frameName>
           </plugin>
-          -->
         </gazebo>
   </xacro:macro>
